Commit message: refactor: run ros2_control on the snapshot core

File: urdf/netft.ros2_control.xacro (robot description, xacro)
@@ -1,5 +1,5 @@
 <?xml version="1.0"?>
 <robot xmlns:xacro="http://www.ros.org/wiki/xacro">
-  <xacro:macro name="netft_ros2_control" params="name sensor_name sensor_ip sensor_port:=49152 counts_per_force:=1000000 counts_per_torque:=1000000 receive_timeout:=0.1 activation_timeout:=2.0 bias_service:=''">
+  <xacro:macro name="netft_ros2_control" params="name sensor_name sensor_ip sensor_port:=49152 http_port:=80 use_sensor_calibration:=true counts_per_force:=1000000 counts_per_torque:=1000000 receive_timeout:=0.1 configuration_connect_timeout:=0.5 configuration_timeout:=1.0 activation_timeout:=2.0 bias_service:=''">
     <ros2_control name="${name}" type="sensor">
       <hardware>
@@ -7,7 +7,11 @@
         <param name="sensor_ip">${sensor_ip}</param>
         <param name="sensor_port">${sensor_port}</param>
+        <param name="http_port">${http_port}</param>
+        <param name="use_sensor_calibration">${use_sensor_calibration}</param>
         <param name="counts_per_force">${counts_per_force}</param>
         <param name="counts_per_torque">${counts_per_torque}</param>
         <param name="receive_timeout">${receive_timeout}</param>
+        <param name="configuration_connect_timeout">${configuration_connect_timeout}</param>
+        <param name="configuration_timeout">${configuration_timeout}</param>
         <param name="activation_timeout">${activation_timeout}</param>
         <xacro:if value="${bias_service != ''}">

Commit message: fix: default ros2 control sensor endpoint

File: urdf/netft.ros2_control.xacro (robot description, xacro)
@@ -1,5 +1,5 @@
 <?xml version="1.0"?>
 <robot xmlns:xacro="http://www.ros.org/wiki/xacro">
-  <xacro:macro name="netft_ros2_control" params="name sensor_name sensor_ip sensor_port:=49152 http_port:=80 use_sensor_calibration:=true counts_per_force:=1000000 counts_per_torque:=1000000 receive_timeout:=0.1 configuration_connect_timeout:=0.5 configuration_timeout:=1.0 activation_timeout:=2.0 bias_service:=''">
+  <xacro:macro name="netft_ros2_control" params="name sensor_name sensor_ip:=192.168.1.1 sensor_port:=49152 http_port:=80 use_sensor_calibration:=true counts_per_force:=1000000 counts_per_torque:=1000000 receive_timeout:=0.1 configuration_connect_timeout:=0.5 configuration_timeout:=1.0 activation_timeout:=2.0 bias_service:=''">
     <ros2_control name="${name}" type="sensor">
       <hardware>

Commit message: Use a private netft-cpp core snapshot (#9)
* Add snapshot core build contract

* core: snapshot netft-cpp v0.1.2

* feat: convert sensor-native samples to SI units

* feat: use sensor calibration by default

* refactor: adapt ROS diagnostics to netft core health

* refactor: run netft_check on the snapshot core

* refactor: run ROS nodes on the snapshot core

* refactor: run ros2_control on the snapshot core

* fix: address ros2_control migration review

* feat: configure automatic sensor calibration in ROS

* fix: default ros2 control sensor endpoint

* refactor: remove the original Net F/T runtime

* docs: explain core provenance and calibration behavior

* release: prepare netft_driver 0.3.0

* fix: address final core migration review

* test: support source trees without git metadata

* chore: remove internal verification report

* fix: support libstdc++ without float from_chars

* fix: hide ros2 control implementation symbols

* test: wait for asynchronous stop command

* docs: clarify compatibility and license boundaries

* test: support Noetic Python 3.8

* test: keep healthy sensor sample observable

* license: adopt Apache-2.0 project-wide

* fix: address final review feedback

File: urdf/netft.ros2_control.xacro (robot description, xacro)
@@ -1,5 +1,5 @@
 <?xml version="1.0"?>
 <robot xmlns:xacro="http://www.ros.org/wiki/xacro">
-  <xacro:macro name="netft_ros2_control" params="name sensor_name sensor_ip sensor_port:=49152 counts_per_force:=1000000 counts_per_torque:=1000000 receive_timeout:=0.1 activation_timeout:=2.0 bias_service:=''">
+  <xacro:macro name="netft_ros2_control" params="name sensor_name sensor_ip:=192.168.1.1 sensor_port:=49152 http_port:=80 use_sensor_calibration:=true counts_per_force:=1000000 counts_per_torque:=1000000 receive_timeout:=0.1 configuration_connect_timeout:=0.5 configuration_timeout:=1.0 activation_timeout:=2.0 bias_service:=''">
     <ros2_control name="${name}" type="sensor">
       <hardware>
@@ -7,7 +7,11 @@
         <param name="sensor_ip">${sensor_ip}</param>
         <param name="sensor_port">${sensor_port}</param>
+        <param name="http_port">${http_port}</param>
+        <param name="use_sensor_calibration">${use_sensor_calibration}</param>
         <param name="counts_per_force">${counts_per_force}</param>
         <param name="counts_per_torque">${counts_per_torque}</param>
         <param name="receive_timeout">${receive_timeout}</param>
+        <param name="configuration_connect_timeout">${configuration_connect_timeout}</param>
+        <param name="configuration_timeout">${configuration_timeout}</param>
         <param name="activation_timeout">${activation_timeout}</param>
         <xacro:if value="${bias_service != ''}">

Commit message: Integrate checked timing and clarify runtime control boundaries

File: urdf/netft.ros2_control.xacro (robot description, xacro)
@@ -1,5 +1,5 @@
 <?xml version="1.0"?>
 <robot xmlns:xacro="http://www.ros.org/wiki/xacro">
-  <xacro:macro name="netft_ros2_control" params="name sensor_name sensor_ip:=192.168.1.1 sensor_port:=49152 http_port:=80 use_sensor_calibration:=true counts_per_force:=1000000 counts_per_torque:=1000000 receive_timeout:=0.1 configuration_connect_timeout:=0.5 configuration_timeout:=1.0 activation_timeout:=2.0 bias_service:=''">
+  <xacro:macro name="netft_ros2_control" params="name sensor_name sensor_ip:=192.168.1.1 sensor_port:=49152 http_port:=80 use_sensor_calibration:=true counts_per_force:=1000000 counts_per_torque:=1000000 receive_timeout:=0.1 configuration_connect_timeout:=0.5 configuration_timeout:=1.0 activation_timeout:=2.0 allow_bias:=true bias_service:=''">
     <ros2_control name="${name}" type="sensor">
       <hardware>
@@ -15,4 +15,5 @@
         <param name="configuration_timeout">${configuration_timeout}</param>
         <param name="activation_timeout">${activation_timeout}</param>
+        <param name="allow_bias">${allow_bias}</param>
         <xacro:if value="${bias_service != ''}">
           <param name="bias_service">${bias_service}</param>
